Commit message: feat(aerial): F450 airframe, hold reward, sim realism, eval tools
Code and configs behind the released model
skydreamer-f450-4.4m-1c-2026-10-17 (config aerial_12in_skydreamer_hold,
Stage 1c, 4.38M steps).

- Airframe: QWinOut F450 kit (1.514 kg est., 10" props, TWR 2.15) from
  a parts table; URDF with legs, prop disks, gimbal; airframe tests.
- Env: ArduPilot-style 400 Hz rate loop, motor lag, latency, estimator
  errors, gusts, drag; ground contact is a crash; mostly-horizontal wind.
- Reward: hold term, ground penalty, rebalanced weights.
- Agent: eval/deploy act with the policy mean; imag_length 32 config.
- Deploy: publish/pull release scripts use the origin fork; NumPy bench
  docs use mean actions.
- Tools: eval_bundle, scripted_hover_pid, plot_trajectories, live_view,
  target_test.

Co-Authored-By: Claude Opus 5.5 <noreply@anthropic.com>
Claude-Session: https://claude.ai/code/session_01MaBregvVTaKdhFMZpbA9ck

File: aerial/assets/cf12in.urdf (robot description, URDF)
Before this commit: robot cf12in, 6 links, 5 joints
Links:
- link base_link: mass 0.8 -> 1.514; geometry collision box size=0.015 0.015 0.14; collision box size=0.015 0.015 0.14

Commit message: feat(aerial): camera/battery-on-top F450, rotor reaction torque, smooth config
Code behind the aerial_12in_skydreamer_smooth run, whose 9.4M-step
checkpoint is the current best Stage 1c policy (30/30, 0.12 m median,
rate-command change 0.36 rad/s vs 3.1 for the previous model).

- Airframe: camera in the gimbal, battery and Orange Pi stacked on top
  -> 1.634 kg, TWR 2.00, inertia 0.0176/0.0183/0.0212; URDF to match.
- Env: rotor reaction torque J*dw/dt on yaw (J = 4.5e-5 kg m^2);
  gym-pybullet-drones only applies the steady drag torque.
- Config aerial_12in_skydreamer_smooth: smooth_coef 0.002 -> 0.05; the
  hold policy chattered (~3 rad/s per 20 ms step) with or without
  sensor noise.
- export_model.py: --step / --ckpt to export a checkpoint other than
  the latest; ckpt_sweep.py evaluates checkpoints across a run.

Co-Authored-By: Claude Opus 5.5 <noreply@anthropic.com>
Claude-Session: https://claude.ai/code/session_01MaBregvVTaKdhFMZpbA9ck

File: aerial/assets/cf12in.urdf (robot description, URDF)
Before this commit: robot cf12in, 6 links, 5 joints
Links:
- link base_link: mass 1.514 -> 1.634
